File: mm_motor_control.kicad_sch (KiCad schematic)
At the start: 0 parts

Commit message: robot
Parts:
- added C10: 10n, symbol Device:C
- added C11: 1n, symbol Device:C
- added C12: 2.2n, symbol Device:C
- added C14: 22n, symbol Device:C_Polarized
- added C9: 22n, symbol Device:C
- added R10: 10k, symbol Device:R
- added R11: 47k, symbol Device:R
- added R12, R13: 330m, symbol Device:R
- added R14, R15: 18k, symbol Device:R
- added U4: STSPIN240, Package_DFN_QFN:VQFN-16-1EP_3x3mm_P0.5mm_EP1.8x1.8mm, symbol Driver_Motor:STSPIN240
Connections:
- net EN: now also R14.1
- net FAULT: now also C10.2, R14.2, U4.13 (EN/FLT)
- net OUT_A1: now also U4.3 (OUTA1)
- net OUT_A2: now also U4.5 (OUTA2)
- net OUT_B1: now also U4.10 (OUTB1)
- net OUT_B2: now also U4.8 (OUTB2)
- net PHASE_A: now also U4.1 (PHA)
- net PHASE_B: now also U4.15 (PHB)
- net PWM_A: now also U4.2 (PWMA)
- net PWM_B: now also U4.16 (PWMB)
- net STBY/RESET: now also C11.1, R15.2, U4.14 (STBY/RESET)
- new net: C9.1, R10.2
- new net: R12.1, U4.9 (SENSEB)
- new net: R10.1, R11.1, U4.12 (TOFF)
- new net: R13.1, U4.4 (SENSEA)
- new net +3.3V: R15.1
- new net +BATT: C12.1, C14.1, U4.6 (VS)
- new net GND: C10.1, C11.2, C12.2, C14.2, C9.2, R11.2, R12.2, R13.2, U4.7 (GND)

Commit message: tp3
Parts:
- removed C14: 22n, symbol Device:C_Polarized
- added C14: 22u, Capacitor_SMD:C_0603_1608Metric, symbol Device:C
- C10: value 10n -> 10u; footprint (none) -> Capacitor_SMD:C_0603_1608Metric
- C11: footprint (none) -> Capacitor_SMD:C_0603_1608Metric
- C12: value 2.2n -> 2.2u; footprint (none) -> Capacitor_SMD:C_0603_1608Metric
- C9: value 22n -> 22u; footprint (none) -> Capacitor_SMD:C_0603_1608Metric
- R10, R11, R12, R13, R14, R15: footprint (none) -> Resistor_SMD:R_0603_1608Metric
Connections:
- net +BATT: now also C14.1
- net GND: now also C14.2
Changed lines of the file:
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@@
+    (stroke (width 0) (type default))
+  )
+  (wire (pts (xy 143.51 66.04) (xy 161.29 66.04))
     (stroke (width 0) (type default))
   )
@@
     (stroke (width 0) (type default))
   )
-  (wire (pts (xy 143.51 66.04) (xy 156.21 66.04))
-    (stroke (width 0) (type default))
-  )
   (wire (pts (xy 80.01 114.3) (xy 88.9 114.3))
     (stroke (width 0) (type default))
@@
   )
   (wire (pts (xy 88.9 114.3) (xy 88.9 115.57))
+    (stroke (width 0) (type default))
+  )
+  (wire (pts (xy 161.29 73.66) (xy 156.21 73.66))
     (stroke (width 0) (type default))
   )
@@
     (effects (font (size 1.27 1.27)) (justify right))
   )
-  (symbol (lib_id "Device:C_Polarized") (at 156.21 69.85 0) (unit 1)
-    (in_bom yes) (on_board yes) (dnp no) (fields_autoplaced)
-    (property "Reference" "C14" (at 160.02 67.691 0)
-      (effects (font (size 1.27 1.27)) (justify left))
-    )
-    (property "Value" "22n" (at 160.02 70.231 0)
-      (effects (font (size 1.27 1.27)) (justify left))
-    )
-    (property "Footprint" "" (at 157.1752 73.66 0)
-      (effects (font (size 1.27 1.27)) hide)
-    )
-    (property "Datasheet" "~" (at 156.21 69.85 0)
-      (effects (font (size 1.27 1.27)) hide)
-    )
-    (pin "1")
-    (pin "2")
-    (instances
-      (project "minimouse"
-        (path "/d8fa4cba-2469-4231-847f-065b6b829f44/0999fad3-9a14-4ede-b729-a71c3dbbdf8e"
-          (reference "C14") (unit 1)
-        )
-      )
-    )
-  )
   (symbol (lib_id "power:+3.3V") (at 88.9 100.33 0) (unit 1)
     (in_bom yes) (on_board yes) (dnp no) (fields_autoplaced)
@@
       (effects (font (size 1.27 1.27)) (justify left))
     )
-    (property "Value" "2.2n" (at 147.32 71.12 0)
-      (effects (font (size 1.27 1.27)) (justify left))
-    )
-    (property "Footprint" "" (at 144.4752 73.66 0)
+    (property "Value" "2.2u" (at 147.32 71.12 0)
+      (effects (font (size 1.27 1.27)) (justify left))
+    )
+    (property "Footprint" "Capacitor_SMD:C_0603_1608Metric" (at 144.4752 73.66 0)
       (effects (font (size 1.27 1.27)) hide)
     )
@@
       (effects (font (size 1.27 1.27)) (justify left))
     )
-    (property "Value" "22n" (at 106.68 123.19 0)
-      (effects (font (size 1.27 1.27)) (justify left))
-    )
-    (property "Footprint" "" (at 103.8352 125.73 0)
+    (property "Value" "22u" (at 106.68 123.19 0)
+      (effects (font (size 1.27 1.27)) (justify left))
+    )
+    (property "Footprint" "Capacitor_SMD:C_0603_1608Metric" (at 103.8352 125.73 0)
       (effects (font (size 1.27 1.27)) hide)
     )
@@
       (effects (font (size 1.27 1.27)) (justify right))
     )
-    (property "Value" "10n" (at 76.2 99.06 0)
+    (property "Value" "10u" (at 76.2 99.06 0)
       (effects (font (size 1.27 1.27)) (justify right))
     )
-    (property "Footprint" "" (at 71.4248 93.98 0)
+    (property "Footprint" "Capacitor_SMD:C_0603_1608Metric" (at 71.4248 93.98 0)
       (effects (font (size 1.27 1.27)) hide)
     )
@@
       (effects (font (size 1.27 1.27)) (justify left))
     )
-    (property "Footprint" "" (at 143.002 100.33 90)
+    (property "Footprint" "Resistor_SMD:R_0603_1608Metric" (at 143.002 100.33 90)
       (effects (font (size 1.27 1.27)) hide)
     )
@@
     )
   )
+  (symbol (lib_id "Device:C") (at 161.29 69.85 0) (unit 1)
+    (in_bom yes) (on_board yes) (dnp no) (fields_autoplaced)
+    (property "Reference" "C14" (at 165.1 68.58 0)
+      (effects (font (size 1.27 1.27)) (justify left))
+    )
+    (property "Value" "22u" (at 165.1 71.12 0)
+      (effects (font (size 1.27 1.27)) (justify left))
+    )
+    (property "Footprint" "Capacitor_SMD:C_0603_1608Metric" (at 162.2552 73.66 0)
+      (effects (font (size 1.27 1.27)) hide)
+    )
+    (property "Datasheet" "~" (at 161.29 69.85 0)
+      (effects (font (size 1.27 1.27)) hide)
+    )
+    (pin "1")
+    (pin "2")
+    (instances
+      (project "minimouse"
+        (path "/d8fa4cba-2469-4231-847f-065b6b829f44/0999fad3-9a14-4ede-b729-a71c3dbbdf8e"
+          (reference "C14") (unit 1)
+        )
+      )
+    )
+  )
   (symbol (lib_id "Device:R") (at 110.49 115.57 0) (unit 1)
     (in_bom yes) (on_board yes) (dnp no) (fields_autoplaced)
@@
       (effects (font (size 1.27 1.27)) (justify left))
     )
-    (property "Footprint" "" (at 108.712 115.57 90)
+    (property "Footprint" "Resistor_SMD:R_0603_1608Metric" (at 108.712 115.57 90)
       (effects (font (size 1.27 1.27)) hide)
     )
@@
       (effects (font (size 1.27 1.27)) (justify left))
     )
-    (property "Footprint" "" (at 87.122 107.95 90)
+    (property "Footprint" "Resistor_SMD:R_0603_1608Metric" (at 87.122 107.95 90)
       (effects (font (size 1.27 1.27)) hide)
     )
@@
       (effects (font (size 1.27 1.27)))
     )
-    (property "Footprint" "" (at 149.86 85.598 90)
+    (property "Footprint" "Resistor_SMD:R_0603_1608Metric" (at 149.86 85.598 90)
       (effects (font (size 1.27 1.27)) hide)
     )
@@
       (effects (font (size 1.27 1.27)) (justify left))
     )
-    (property "Footprint" "" (at 89.8652 123.19 0)
+    (property "Footprint" "Capacitor_SMD:C_0603_1608Metric" (at 89.8652 123.19 0)
       (effects (font (size 1.27 1.27)) hide)
     )
@@
       (effects (font (size 1.27 1.27)) (justify left))
     )
-    (property "Footprint" "" (at 101.092 110.49 90)
+    (property "Footprint" "Resistor_SMD:R_0603_1608Metric" (at 101.092 110.49 90)
       (effects (font (size 1.27 1.27)) hide)
     )
@@
       (effects (font (size 1.27 1.27)) (justify left))
     )
-    (property "Footprint" "" (at 66.04 95.758 90)
-      (effects (font (size 1.27 1.27)) hide)
-    )
+    (property "Footprint" "Resistor_SMD:R_0603_1608Metric" (at 66.04 95.758 90)
+      (effects (font (size 1.27 1.27)) hide)
+    )
