File: mm_power.kicad_sch (KiCad schematic)
At the start: 1 part, among them J5 Conn_01x02

Commit message: robot
Parts:
- added C7, C8: 1uF, symbol Device:C
- added U5: LP5907MFX-3.3, Package_TO_SOT_SMD:SOT-23-5, symbol Regulator_Linear:LP5907MFX-3.3
Connections:
- net +BATT: now also C7.2, U5.1 (IN), U5.3 (EN)
- net GND: now also C7.1, C8.1, U5.2 (GND)
- new net +3.3V: C8.2, U5.5 (OUT)

Commit message: tp3
Parts:
- C7, C8: footprint (none) -> Capacitor_SMD:C_0603_1608Metric
Changed lines of the file:
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@@
       (effects (font (size 1.27 1.27)) (justify left))
     )
-    (property "Footprint" "" (at 141.2748 91.44 0)
+    (property "Footprint" "Capacitor_SMD:C_0603_1608Metric" (at 141.2748 91.44 0)
       (effects (font (size 1.27 1.27)) hide)
     )
@@
       (effects (font (size 1.27 1.27)) (justify left))
     )
-    (property "Footprint" "" (at 109.5248 91.44 0)
+    (property "Footprint" "Capacitor_SMD:C_0603_1608Metric" (at 109.5248 91.44 0)
       (effects (font (size 1.27 1.27)) hide)
     )
