File: minimouse.kicad_pcb (KiCad board)
At the start: 2 copper layers, 90 x 85 mm, 22 parts, among them J1 Conn_ARM_JTAG_SWD_10, J5 Conn_01x02, M1 N20_encoder, M2 N20_encoder, U1 STM32F030C8Tx, U4 HC-SR04

Commit message: tp3
Parts:
- added C10: 10u, Capacitor_SMD:C_0603_1608Metric, F.Cu at (152.5, 96.5)
- added C11: 1n, Capacitor_SMD:C_0603_1608Metric, F.Cu at (148.0, 96.5)
- added C12: 2.2u, Capacitor_SMD:C_0603_1608Metric, F.Cu at (150.0, 105.4)
- added C14: 22u, Capacitor_SMD:C_0603_1608Metric, F.Cu at (149.9, 107.1)
- added C7: 1uF, Capacitor_SMD:C_0603_1608Metric, F.Cu at (131.3, 90.8)
- added C8: 1uF, Capacitor_SMD:C_0603_1608Metric, F.Cu at (145.2, 76.7)
- added C9: 22u, Capacitor_SMD:C_0603_1608Metric, F.Cu at (158.0, 99.6)
- added J2: Conn_01x06, Connector_PinHeader_2.54mm:PinHeader_1x06_P2.54mm_Vertical, F.Cu at (162.6, 104.3)
- added J3: Conn_01x04, Connector_PinHeader_2.54mm:PinHeader_1x04_P2.54mm_Vertical, F.Cu at (157.6, 65.0)
- added J4: Conn_01x06, Connector_PinHeader_2.54mm:PinHeader_1x06_P2.54mm_Vertical, F.Cu at (136.1, 104.3)
- added R10: 10k, Resistor_SMD:R_0603_1608Metric, F.Cu at (155.0, 99.6)
- added R11: 47k, Resistor_SMD:R_0603_1608Metric, F.Cu at (155.0, 101.1)
- added R12: 330m, Resistor_SMD:R_0603_1608Metric, F.Cu at (155.0, 102.6)
- added R13: 330m, Resistor_SMD:R_0603_1608Metric, F.Cu at (145.1, 103.3)
- added R14: 18k, Resistor_SMD:R_0603_1608Metric, F.Cu at (151.0, 96.5)
- added R15: 18k, Resistor_SMD:R_0603_1608Metric, F.Cu at (149.5, 96.5)
- added U2: HC-SR04, minimouse:HC-SR04, F.Cu at (150.0, 64.1)
- added U5: LP5907MFX-3.3, Package_TO_SOT_SMD:SOT-23-5, F.Cu at (129.3, 85.2)
- U4: value HC-SR04 -> STSPIN240; footprint minimouse:HC-SR04 -> Package_DFN_QFN:VQFN-16-1EP_3x3mm_P0.5mm_EP1.8x1.8mm
- moved U4 31.9 mm to (150.0, 101.0)
- moved C1 27.2 mm to (166.5, 78.8), turned to 90 degrees
- moved C5 22.1 mm to (143.2, 78.4)
- moved C2 19.4 mm to (125.7, 82.7), turned to 180 degrees
- moved BOOT0 15.3 mm to (143.8, 70.7)
- moved R1 11.0 mm to (149.7, 70.1)
- moved C6 9.95 mm to (137.9, 74.6), turned to -90 degrees
- moved R4 9.91 mm to (147.8, 90.1)
- moved R5 9.91 mm to (149.3, 90.1)
- moved R3 9.90 mm to (146.3, 90.1)
- moved R6 9.32 mm to (150.8, 90.1)
- moved R7 9.32 mm to (152.3, 90.1)
- moved C4 9.18 mm to (154.6, 85.7)
- moved U1 8.38 mm to (149.9, 81.2)
- moved R9 7.63 mm to (147.5, 73.5)
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Connections:
- R8 pad 1: /mcu/UART1_TX -> /external_uart/EXT_UART_RX
- U1 pad 43: /mcu/UART1_RX -> /external_uart/EXT_UART_TX
- U4 pad 1: GND -> /mcu/OUT_A4
- U4 pad 2: /mcu/OUT_B9 -> /mcu/TIM15_CH1
- U4 pad 3: Net-(U4-ECHO) -> /motorB/MA
- U4 pad 4: +3V3 -> Net-(U4-SENSEA)
Routing:
- net GND: track 0.00 -> 173.1 mm, vias 0 -> 6
- net +BATT: track 0.00 -> 129.4 mm, vias 0 -> 2
- net +3.3V: track 0.00 -> 44.4 mm, vias 0 -> 2
- net /motorA/MB: track 0.00 -> 24.1 mm, vias 0 -> 2
- net /mcu/TIM3_CH1: track 0.00 -> 22.4 mm, vias 0 -> 2
- net /mcu/TIM2_CH1: track 0.00 -> 22.2 mm, vias 0 -> 2
- net /mcu/~{RESET}: track 0.00 -> 22.1 mm, vias 0 -> 2
- net /motorB/MB: track 0.00 -> 21.0 mm
- net /mcu/TIM3_CH2: track 0.00 -> 19.6 mm, vias 0 -> 2
- net /mcu/TIM2_CH2: track 0.00 -> 18.2 mm, vias 0 -> 2
- net /mcu/TIM8_CH2: track 0.00 -> 16.7 mm, vias 0 -> 2
- net /external_uart/EXT_UART_TX: track 0.00 -> 13.8 mm
- net /motorB/MA: track 0.00 -> 12.7 mm, vias 0 -> 2
- net /mcu/SWO: track 0.00 -> 12.7 mm
- net /mcu/OUT_A4: track 0.00 -> 12.4 mm, vias 0 -> 2
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
Commit message: tp4
Parts:
- moved C7 7.33 mm to (125.8, 85.9), turned to -90 degrees
- moved C2 6.62 mm to (132.3, 83.0), turned to 90 degrees
- moved C1 5.02 mm to (162.2, 81.4), turned to 180 degrees
- moved BOOT0 4.64 mm to (147.9, 68.6)
- moved C6 4.63 mm to (136.2, 78.9), turned to 90 degrees
- moved R13 2.48 mm to (143.1, 101.9), turned to 180 degrees
- moved C3 1.40 mm to (142.3, 81.1)
- moved R12 0.10 mm to (155.0, 102.7)
Routing:
- net GND: track 173.1 -> 26.3 mm, vias 6 -> 22
- net +3.3V: track 44.4 -> 71.1 mm
- net /mcu/IN_B2: track 3.76 -> 19.6 mm
- net /mcu/OUT_A5: track 0.00 -> 11.9 mm
- net /mcu/OUT_B0: track 3.98 -> 13.1 mm
- net /mcu/OUT_B1: track 0.00 -> 5.32 mm
- net Net-(U4-SENSEA): track 0.00 -> 4.64 mm
- net /mcu/OUT_B9: track 9.10 -> 12.6 mm
- net Net-(U4-SENSEB): track 0.00 -> 3.13 mm
- net +BATT: track 129.4 -> 132.3 mm, vias 2 -> 0
- net /motorB/MB: track 21.0 -> 23.3 mm
- net /mcu/BOOT0: track 12.1 -> 10.5 mm, vias 2 -> 0
- net /mcu/TIM2_CH2: track 18.2 -> 19.7 mm
- net /mcu/TIM3_CH1: track 22.4 -> 23.5 mm
- net /mcu/TIM15_CH1: track 12.1 -> 13.0 mm
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- added copper zone on B.Cu, net GND
